File: licznik.kicad_pcb (KiCad board)
At the start: 2 copper layers, 54.6 x 45.7 mm, 32 parts, among them J1 Display, J2 Micro_SD_Card_Det, J3 Serial CS1, J4 Serial CS2, SW1 Wheel, SW2 Crank, SW3 Backlight, SW4 Right, SW5 Select, SW6 Left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

Commit message: Fix track moving over a hole
Routing:
- net GND: track 195.6 -> 194.7 mm
Changed lines of the file:
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@@
     (thickness 1.6)
     (drawings 16)
-    (tracks 264)
+    (tracks 267)
     (zones 0)
     (modules 32)
@@
   )
   (layers
-    (0 F.Cu signal hide)
+    (0 F.Cu signal)
     (31 B.Cu signal)
     (32 B.Adhes user)
@@
     (34 B.Paste user)
     (35 F.Paste user)
-    (36 B.SilkS user)
+    (36 B.SilkS user hide)
     (37 F.SilkS user)
     (38 B.Mask user)
@@
   (segment (start 38.68 189.615622) (end 38.68 196.115622) (width 0.25) (layer F.Cu) (net 24))
   (segment (start 66.04 191.985622) (end 66.04 190.885622) (width 0.25) (layer F.Cu) (net 24))
-  (segment (start 40.005001 197.440623) (end 60.584999 197.440623) (width 0.25) (layer F.Cu) (net 24))
-  (segment (start 38.68 196.115622) (end 40.005001 197.440623) (width 0.25) (layer F.Cu) (net 24))
   (segment (start 39.679999 186.955621) (end 38.68 185.955622) (width 0.25) (layer F.Cu) (net 24))
   (segment (start 40.005001 187.280623) (end 39.679999 186.955621) (width 0.25) (layer F.Cu) (net 24))
@@
   (segment (start 72.39 191.985622) (end 72.314999 192.060623) (width 0.25) (layer F.Cu) (net 24))
   (segment (start 72.39 190.885622) (end 72.39 191.985622) (width 0.25) (layer F.Cu) (net 24))
-  (segment (start 59.69 190.284378) (end 63.715622 194.31) (width 0.25) (layer F.Cu) (net 24))
   (segment (start 59.69 189.23) (end 59.69 190.284378) (width 0.25) (layer F.Cu) (net 24))
-  (segment (start 60.584999 197.440623) (end 63.715622 194.31) (width 0.25) (layer F.Cu) (net 24))
   (segment (start 63.715622 194.31) (end 66.04 191.985622) (width 0.25) (layer F.Cu) (net 24))
   (segment (start 66.04 190.885622) (end 66.04 187.96) (width 0.25) (layer F.Cu) (net 24))
@@
   (segment (start 67.31 180.725622) (end 66.04 181.995622) (width 2) (layer B.Cu) (net 24))
   (segment (start 67.31 172.72) (end 67.31 180.725622) (width 2) (layer B.Cu) (net 24))
+  (segment (start 60.744378 194.31) (end 62.23 192.824378) (width 0.25) (layer F.Cu) (net 24))
+  (segment (start 62.23 192.824378) (end 63.715622 194.31) (width 0.25) (layer F.Cu) (net 24))
+  (segment (start 59.69 190.284378) (end 62.23 192.824378) (width 0.25) (layer F.Cu) (net 24))
+  (segment (start 38.68 196.115622) (end 40.005001 197.440623) (width 0.25) (layer F.Cu) (net 24))
+  (segment (start 40.005001 197.440623) (end 45.713375 197.440623) (width 0.25) (layer F.Cu) (net 24))
+  (segment (start 45.713375 197.440623) (end 48.843998 194.31) (width 0.25) (layer F.Cu) (net 24))
+  (segment (start 48.843998 194.31) (end 60.744378 194.31) (width 0.25) (layer F.Cu) (net 24))
   (segment (start 53.34 165.655622) (end 53.34 166.755622) (width 0.25) (layer F.Cu) (net 25))
   (segment (start 60.659999 158.335623) (end 53.34 165.655622) (width 0.25) (layer F.Cu) (net 25))

Commit message: Marked version 0.9.1
Parts:
- moved logo 2.84 mm to (53.3, 186.7), turned to 180 degrees
- moved REF** 1.80 mm to (52.1, 174.0), turned to 180 degrees
Other:
- board text added: "v0.9.1"
Changed lines of the file:
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@@
   (general
     (thickness 1.6)
-    (drawings 16)
+    (drawings 18)
     (tracks 267)
     (zones 0)
@@
     (34 B.Paste user)
     (35 F.Paste user)
-    (36 B.SilkS user hide)
+    (36 B.SilkS user)
     (37 F.SilkS user)
     (38 B.Mask user)
@@
     (visible_elements FFFFFF7F)
     (pcbplotparams
-      (layerselection 0x00030_80000001)
+      (layerselection 0x010f0_ffffffff)
       (usegerberextensions false)
-      (usegerberattributes false)
+      (usegerberattributes true)
       (usegerberadvancedattributes false)
-      (creategerberjobfile false)
+      (creategerberjobfile true)
       (excludeedgelayer true)
       (linewidth 0.100000)
@@
       (plotinvisibletext false)
       (padsonsilk false)
-      (subtractmaskfromsilk false)
+      (subtractmaskfromsilk true)
       (outputformat 1)
       (mirror false)
-      (drillshape 1)
+      (drillshape 0)
       (scaleselection 1)
-      (outputdirectory ""))
+      (outputdirectory "/home/rhn/play/licznik_compact/gerber_prototypy/"))
   )
   (net 0 "")
@@
   )
   (module Symbol:OSHW-Logo2_7.3x6mm_SilkScreen (layer B.Cu)
-    (at 53.34 175.26)
+    (at 52.07 173.99 180)
     (descr "Open Source Hardware Symbol")
     (tags "Logo Symbol OSHW")
     (attr virtual)
-    (fp_text reference REF** (at 0 0) (layer B.SilkS) hide
+    (fp_text reference REF** (at 0 0 180) (layer B.SilkS) hide
       (effects (font (size 1 1) (thickness 0.15)) (justify mirror))
     )
-    (fp_text value OSHW-Logo2_7.3x6mm_SilkScreen (at 0.75 0) (layer B.Fab) hide
+    (fp_text value OSHW-Logo2_7.3x6mm_SilkScreen (at 0.75 0 180) (layer B.Fab) hide
       (effects (font (size 1 1) (thickness 0.15)) (justify mirror))
     )
@@
   )
   (module Licznik:logo_ss (layer B.Cu)
-    (at 54.61 189.23)
+    (at 53.34 186.69 180)
     (descr "Imported from /home/rhn/mnt/gateway/play/jazda/logo_text_kicad.svg")
     (tags svg2mod)
     (attr smd)
-    (fp_text reference logo (at 0 11.9938) (layer B.SilkS) hide
+    (fp_text reference logo (at 0 11.9938 180) (layer B.SilkS) hide
       (effects (font (size 1.524 1.524) (thickness 0.3048)) (justify mirror))
     )
-    (fp_text value G*** (at 0 -11.9938) (layer B.SilkS) hide
+    (fp_text value G*** (at 0 -11.9938 180) (layer B.SilkS) hide
       (effects (font (size 1.524 1.524) (thickness 0.3048)) (justify mirror))
     )
@@
       (xy 5.473769 2.362728) (xy 5.272436 2.49054) (xy 5.058595 2.60173) (xy 5.169915 2.84196)) (layer B.SilkS) (width 0))
   )
+  (gr_text v0.9.1 (at 53.34 196.85) (layer B.SilkS)
+    (effects (font (size 1 1) (thickness 0.2)) (justify mirror))
+  )
+  (gr_text v0.9.1 (at 53.34 198.12) (layer F.SilkS)
+    (effects (font (size 1 1) (thickness 0.2)))
+  )
   (gr_text Wheel (at 71.12 199.39) (layer B.SilkS)
     (effects (font (size 1.5 1.5) (thickness 0.3)) (justify mirror))
@@
   (segment (start 43.18 196.115622) (end 43.18 189.615622) (width 0.25) (layer F.Cu) (net 14))
   (segment (start 45.615622 187.18) (end 43.18 189.615622) (width 0.25) (layer F.Cu) (net 14))
-  (segment (start 59.69 187.18) (end 45.615622 187.18) (width 0.25) (layer F.Cu) (net 14))
   (segment (start 73.740622 179.455622) (end 73.66 179.375) (width 0.25) (layer F.Cu) (net 14))
   (segment (start 76.2 179.455622) (end 73.740622 179.455622) (width 0.25) (layer F.Cu) (net 14))
@@
   (segment (start 59.69 187.18) (end 63.01 187.18) (width 0.25) (layer F.Cu) (net 14))
   (segment (start 63.01 187.18) (end 69.388388 180.801612) (width 0.25) (layer F.Cu) (net 14))
+  (segment (start 59.69 187.18) (end 45.615622 187.18) (width 0.25) (layer F.Cu) (net 14))
   (segment (start 76.119378 181.915) (end 76.2 181.995622) (width 0.25) (layer F.Cu) (net 15))
   (segment (start 63.5 188.45) (end 63.99 187.96) (width 0.25) (layer F.Cu) (net 15))
