File: kicad/licznik.sch (KiCad schematic (older format))
At the start: 24 parts, among them J1 Display, J2 Micro_SD_Card_Det, J3 Serial CS1, J4 Serial CS2, SW1 Wheel, SW2 Crank, SW3 Backlight, SW4 Right, SW5 Select, SW6 Left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

Commit message: Allowed kicad to fix missing libraries
Parts:
- SW3, SW4, SW5, SW6: symbol New_Library:SW_CONN_x6 -> licznik-rescue:SW_CONN_x6-New_Library
Changed lines of the file:
@@
 Connection ~ 5650 4350
 $Comp
-L New_Library:SW_CONN_x6 SW3
+L licznik-rescue:SW_CONN_x6-New_Library SW3
 U 1 1 5BED9366
 P 6000 4150
@@
 	5650 4350 5900 4350
 $Comp
-L New_Library:SW_CONN_x6 SW4
+L licznik-rescue:SW_CONN_x6-New_Library SW4
 U 1 1 5BEDBF4F
 P 6450 4150
@@
 $EndComp
 $Comp
-L New_Library:SW_CONN_x6 SW5
+L licznik-rescue:SW_CONN_x6-New_Library SW5
 U 1 1 5BEDBF99
 P 6950 4150
@@
 $EndComp
 $Comp
-L New_Library:SW_CONN_x6 SW6
+L licznik-rescue:SW_CONN_x6-New_Library SW6
 U 1 1 5BEDC017
 P 7500 4150

Commit message: PCB: Use optional RTC capacitor
Parts:
- added C7: 100µF, Capacitor_SMD:C_1210_3225Metric_Pad1.42x2.65mm_HandSolder, symbol Device:C
Connections:
- net +BATT: now also C7.1
- net GND: now also C7.2
Changed lines of the file:
@@
 Connection ~ 3500 1000
-Wire Wire Line
-	2400 2700 2400 3800
 Wire Wire Line
 	2400 3800 3400 3800
@@
 Connection ~ 2400 1300
 Wire Wire Line
-	2400 1300 2400 2400
+	2400 1300 2400 2250
 Wire Wire Line
 	5000 3850 5000 4050
@@
 	1    0    0    -1
 $EndComp
+Wire Wire Line
+	2400 2250 2100 2250
+Connection ~ 2400 2250
+Wire Wire Line
+	2400 2250 2400 2400
+$Comp
+L Device:C C7
+U 1 1 5C1FFB03
+P 2100 2550
+F 0 "C7" H 2215 2596 50  0000 L CNN
+F 1 "100µF" H 2215 2505 50  0000 L CNN
+F 2 "Capacitor_SMD:C_1210_3225Metric_Pad1.42x2.65mm_HandSolder" H 2138 2400 50  0001 C CNN
+F 3 "~" H 2100 2550 50  0001 C CNN
+	1    2100 2550
+	1    0    0    -1
+$EndComp
+Wire Wire Line
+	2400 2700 2400 2800
+Wire Wire Line
+	2100 2250 2100 2400
+Wire Wire Line
+	2100 2700 2100 2800
+Wire Wire Line
+	2100 2800 2400 2800
+Connection ~ 2400 2800
+Wire Wire Line
+	2400 2800 2400 3800
 $EndSCHEMATC

Commit message: Schematic: Added comments
Parts:
- BT1: value 2xAA (2.8V) -> 2xAA (2.4V)
Other:
- note added: "RTC backup capacitor. Optional.\nValue not established - no current usage estimate yet."
- note added: "TODO: Use the display SPI bus for all peripherals."
Changed lines of the file:
@@
 P 2400 2600
 F 0 "BT1" H 2518 2696 50  0000 L CNN
-F 1 "2xAA (2.8V)" H 2518 2605 50  0000 L CNN
+F 1 "2xAA (2.4V)" H 2518 2605 50  0000 L CNN
 F 2 "Connector_PinHeader_2.54mm:PinHeader_1x02_P2.54mm_Vertical" V 2400 2660 50  0001 C CNN
 F 3 "~" V 2400 2660 50  0001 C CNN
@@
 Wire Wire Line
 	2400 2800 2400 3800
+Text Notes -150 2600 0    50   ~ 0
+RTC backup capacitor. Optional.\nValue not established - no current usage estimate yet.
+Text Notes 5050 2350 0    50   ~ 0
+TODO: Use the display SPI bus for all peripherals.
 $EndSCHEMATC
